File: ESP32-A1S-Header.kicad_pcb (KiCad board)
At the start: 2 copper layers, 36.8 x 45 mm, 3 parts, among them J1 Conn_01x16_Male, J2 Conn_01x16_Male, U1 ESP32-A1S

Commit message: gg
Routing:
- net Net-(U1-Pad16): track 9.56 -> 10.1 mm
Changed lines of the file:
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@@
   (segment (start 126.746 105.664) (end 125.73 106.68) (width 0.5) (layer "F.Cu") (net 14))
   (segment (start 128.896 102.498) (end 126.746 104.648) (width 0.5) (layer "F.Cu") (net 14))
-  (segment (start 130.166 103.768) (end 127.508 106.426) (width 0.5) (layer "F.Cu") (net 15))
+  (segment (start 127.508 108.458) (end 126.746 109.22) (width 0.5) (layer "F.Cu") (net 15))
+  (segment (start 131.081 103.768) (end 129.277 103.768) (width 0.5) (layer "F.Cu") (net 15))
+  (segment (start 129.277 103.768) (end 127.508 105.537) (width 0.5) (layer "F.Cu") (net 15))
+  (segment (start 127.508 105.537) (end 127.508 108.458) (width 0.5) (layer "F.Cu") (net 15))
   (segment (start 126.746 109.22) (end 124.968 109.22) (width 0.5) (layer "F.Cu") (net 15))
-  (segment (start 127.508 106.426) (end 127.508 108.458) (width 0.5) (layer "F.Cu") (net 15))
-  (segment (start 127.508 108.458) (end 126.746 109.22) (width 0.5) (layer "F.Cu") (net 15))
-  (segment (start 131.081 103.768) (end 130.166 103.768) (width 0.5) (layer "F.Cu") (net 15))
   (segment (start 128.27 106.68) (end 128.27 110.744) (width 0.5) (layer "F.Cu") (net 16))
   (segment (start 127.254 111.76) (end 124.968 111.76) (width 0.5) (layer "F.Cu") (net 16))
@@
   (segment (start 129.912 106.308) (end 129.286 106.934) (width 0.5) (layer "F.Cu") (net 17))
   (segment (start 152.4 77.216) (end 153.416 76.2) (width 0.5) (layer "F.Cu") (net 18))
+  (segment (start 152.4 85.423) (end 151.835 85.988) (width 0.5) (layer "F.Cu") (net 18))
   (segment (start 153.416 76.2) (end 157 76.2) (width 0.5) (layer "F.Cu") (net 18))
-  (segment (start 150.855 85.988) (end 152.01 85.988) (width 0.5) (layer "F.Cu") (net 18))
-  (segment (start 152.4 85.598) (end 152.4 77.216) (width 0.5) (layer "F.Cu") (net 18))
-  (segment (start 152.01 85.988) (end 152.4 85.598) (width 0.5) (layer "F.Cu") (net 18))
-  (segment (start 153.162 80.264) (end 154.686 78.74) (width 0.5) (layer "F.Cu") (net 19))
-  (segment (start 154.686 78.74) (end 157 78.74) (width 0.5) (layer "F.Cu") (net 19))
-  (segment (start 150.855 87.258) (end 152.01 87.258) (width 0.5) (layer "F.Cu") (net 19))
-  (segment (start 153.162 86.106) (end 153.162 80.264) (width 0.5) (layer "F.Cu") (net 19))
-  (segment (start 152.01 87.258) (end 153.162 86.106) (width 0.5) (layer "F.Cu") (net 19))
+  (segment (start 152.4 77.216) (end 152.4 85.423) (width 0.5) (layer "F.Cu") (net 18))
+  (segment (start 151.835 85.988) (end 150.855 85.988) (width 0.5) (layer "F.Cu") (net 18))
+  (segment (start 153.162 80.264) (end 153.162 86.13205) (width 0.5) (layer "F.Cu") (net 19))
+  (segment (start 152.03605 87.258) (end 150.855 87.258) (width 0.5) (layer "F.Cu") (net 19))
+  (segment (start 153.162 86.13205) (end 152.03605 87.258) (width 0.5) (layer "F.Cu") (net 19))
+  (segment (start 154.686 78.74) (end 153.162 80.264) (width 0.5) (layer "F.Cu") (net 19))
+  (segment (start 157 78.74) (end 154.686 78.74) (width 0.5) (layer "F.Cu") (net 19))
   (segment (start 154.178 86.106) (end 154.178 81.788) (width 0.5) (layer "F.Cu") (net 20))
   (segment (start 154.686 81.28) (end 157 81.28) (width 0.5) (layer "F.Cu") (net 20))
@@
   (segment (start 151.756 89.798) (end 155.194 86.36) (width 0.5) (layer "F.Cu") (net 21))
   (segment (start 155.702 83.82) (end 157 83.82) (width 0.5) (layer "F.Cu") (net 21))
+  (segment (start 152.292 91.068) (end 150.855 91.068) (width 0.5) (layer "F.Cu") (net 22))
   (segment (start 150.855 91.165) (end 150.876 91.186) (width 0.5) (layer "F.Cu") (net 22))
   (segment (start 150.855 91.068) (end 150.855 91.165) (width 0.5) (layer "F.Cu") (net 22))
-  (segment (start 153.67 89.154) (end 154.206 89.154) (width 0.5) (layer "F.Cu") (net 22))
-  (segment (start 150.876 91.186) (end 151.638 91.186) (width 0.5) (layer "F.Cu") (net 22))
-  (segment (start 151.638 91.186) (end 153.67 89.154) (width 0.5) (layer "F.Cu") (net 22))
-  (segment (start 154.206 89.154) (end 157 86.36) (width 0.5) (layer "F.Cu") (net 22))
-  (segment (start 155.984 89.916) (end 157 88.9) (width 0.5) (layer "F.Cu") (net 23))
-  (segment (start 154.432 89.916) (end 155.984 89.916) (width 0.5) (layer "F.Cu") (net 23))
-  (segment (start 150.855 92.338) (end 152.01 92.338) (width 0.5) (layer "F.Cu") (net 23))
-  (segment (start 152.01 92.338) (end 154.432 89.916) (width 0.5) (layer "F.Cu") (net 23))
-  (segment (start 152.772 93.608) (end 154.94 91.44) (width 0.5) (layer "F.Cu") (net 24))
-  (segment (start 150.855 93.608) (end 152.772 93.608) (width 0.5) (layer "F.Cu") (net 24))
-  (segment (start 154.94 91.44) (end 157 91.44) (width 0.5) (layer "F.Cu") (net 24))
+  (segment (start 157 86.36) (end 152.292 91.068) (width 0.5) (layer "F.Cu") (net 22))
+  (segment (start 157 88.9) (end 155.73 90.17) (width 0.5) (layer "F.Cu") (net 23))
+  (segment (start 152.772 92.338) (end 150.855 92.338) (width 0.5) (layer "F.Cu") (net 23))
+  (segment (start 155.73 90.17) (end 155.575 90.17) (width 0.5) (layer "F.Cu") (net 23))
+  (segment (start 153.67 92.075) (end 153.035 92.075) (width 0.5) (layer "F.Cu") (net 23))
+  (segment (start 155.575 90.17) (end 153.67 92.075) (width 0.5) (layer "F.Cu") (net 23))
+  (segment (start 153.035 92.075) (end 152.772 92.338) (width 0.5) (layer "F.Cu") (net 23))
+  (segment (start 157 91.44) (end 155.73 92.71) (width 0.5) (layer "F.Cu") (net 24))
+  (segment (start 155.73 92.71) (end 154.94 92.71) (width 0.5) (layer "F.Cu") (net 24))
+  (segment (start 154.94 92.71) (end 154.042 93.608) (width 0.5) (layer "F.Cu") (net 24))
+  (segment (start 154.042 93.608) (end 150.855 93.608) (width 0.5) (layer "F.Cu") (net 24))
   (segment (start 155.194 93.98) (end 157 93.98) (width 0.5) (layer "F.Cu") (net 25))
   (segment (start 150.855 94.878) (end 154.296 94.878) (width 0.5) (layer "F.Cu") (net 25))
@@
   (segment (start 154.568 97.418) (end 155.194 98.044) (width 0.5) (layer "F.Cu") (net 27))
   (segment (start 150.855 97.418) (end 154.568 97.418) (width 0.5) (layer "F.Cu") (net 27))
-  (segment (start 154.178 99.314) (end 154.714 99.314) (width 0.5) (layer "F.Cu") (net 28))
-  (segment (start 153.552 98.688) (end 154.178 99.314) (width 0.5) (layer "F.Cu") (net 28))
-  (segment (start 150.855 98.688) (end 153.552 98.688) (width 0.5) (layer "F.Cu") (net 28))
-  (segment (start 154.714 99.314) (end 157 101.6) (width 0.5) (layer "F.Cu") (net 28))
+  (segment (start 150.855 98.688) (end 152.663 98.688) (width 0.5) (layer "F.Cu") (net 28))
+  (segment (start 152.663 98.688) (end 155.575 101.6) (width 0.5) (layer "F.Cu") (net 28))
+  (segment (start 155.575 101.6) (end 157 101.6) (width 0.5) (layer "F.Cu") (net 28))
   (segment (start 152.282 99.958) (end 153.416 101.092) (width 0.5) (layer "F.Cu") (net 29))
   (segment (start 155.448 104.14) (end 157 104.14) (width 0.5) (layer "F.Cu") (net 29))
